File: esp32_2/version2/version2.kicad_sch (KiCad schematic)
At the start: 29 parts, among them J1 USB_C_Receptacle_USB2.0_16P, J2 Conn_01x08_Pin, J3 Conn_01x08_Pin, SW1 SW_Push, SW2 SW_Push, U1 USBLC6-2SC6, U2 AP2112K-3.3, U3 ESP32-C3-WROOM-02, Y1 Crystal

Commit message: added copper fill vbus
Parts:
- C6: footprint Capacitor_SMD:C_0805_2012Metric -> Capacitor_SMD:C_0201_0603Metric
Changed lines of the file:
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@@
 			)
 		)
-		(property "Footprint" "Capacitor_SMD:C_0805_2012Metric"
+		(property "Footprint" "Capacitor_SMD:C_0201_0603Metric"
 			(at 84.7852 154.94 0)
 			(hide yes)

Commit message: i feel stupid because the reason everything was breaking because i added an extra gnd pin in my schematic when i wasn't supposed to
Connections:
- net GND: no longer C10.1, J2.8 (Pin_8), R5.1, R6.1, R7.1, SW1.2, SW2.2, U3.8 (IO9)
- new net: R5.1, R6.1, SW1.2
- new net IO9: C10.1, J2.8 (Pin_8), R7.1, SW2.2, U3.8 (IO9)
Changed lines of the file:
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@@
 	)
 	(junction
-		(at 166.37 196.85)
-		(diameter 0)
-		(color 0 0 0 0)
-	)
-	(junction
 		(at 180.34 196.85)
 		(diameter 0)
@@
 	)
 	(junction
-		(at 166.37 154.94)
-		(diameter 0)
-		(color 0 0 0 0)
-	)
-	(junction
 		(at 195.58 154.94)
 		(diameter 0)
@@
 	(wire
 		(pts
-			(xy 162.56 154.94) (xy 166.37 154.94)
+			(xy 162.56 154.94) (xy 180.34 154.94)
 		)
 		(stroke
@@
 	(wire
 		(pts
-			(xy 166.37 154.94) (xy 180.34 154.94)
-		)
-		(stroke
-			(width 0)
-			(type default)
-		)
-	)
-	(wire
-		(pts
 			(xy 152.4 154.94) (xy 147.32 154.94)
 		)
@@
 	(wire
 		(pts
-			(xy 166.37 154.94) (xy 166.37 158.75)
-		)
-		(stroke
-			(width 0)
-			(type default)
-		)
-	)
-	(wire
-		(pts
 			(xy 71.12 121.92) (xy 71.12 123.19)
 		)
@@
 	(wire
 		(pts
-			(xy 162.56 196.85) (xy 166.37 196.85)
-		)
-		(stroke
-			(width 0)
-			(type default)
-		)
-	)
-	(wire
-		(pts
 			(xy 31.75 187.96) (xy 36.83 187.96)
 		)
@@
 	(wire
 		(pts
-			(xy 166.37 196.85) (xy 166.37 200.66)
-		)
-		(stroke
-			(width 0)
-			(type default)
-		)
-	)
-	(wire
-		(pts
 			(xy 73.66 186.69) (xy 81.28 186.69)
 		)
@@
 	(wire
 		(pts
-			(xy 166.37 196.85) (xy 180.34 196.85)
+			(xy 162.56 196.85) (xy 180.34 196.85)
 		)
 		(stroke
@@
 	)
 	(symbol
-		(lib_id "power:GND")
-		(at 166.37 158.75 0)
-		(unit 1)
-		(body_style 1)
-		(exclude_from_sim no)
-		(in_bom yes)
-		(on_board yes)
-		(in_pos_files yes)
-		(dnp no)
-		(fields_autoplaced yes)
-		(property "Reference" "#PWR019"
-			(at 166.37 165.1 0)
-			(hide yes)
-			(show_name no)
-			(do_not_autoplace no)
-			(effects
-				(font
-					(size 1.27 1.27)
-				)
-			)
-		)
-		(property "Value" "GND"
-			(at 166.37 163.83 0)
-			(show_name no)
-			(do_not_autoplace no)
-			(effects
-				(font
-					(size 1.27 1.27)
-				)
-			)
-		)
-		(property "Footprint" ""
-			(at 166.37 158.75 0)
-			(hide yes)
-			(show_name no)
-			(do_not_autoplace no)
-			(effects
-				(font
-					(size 1.27 1.27)
-				)
-			)
-		)
-		(property "Datasheet" ""
-			(at 166.37 158.75 0)
-			(hide yes)
-			(show_name no)
-			(do_not_autoplace no)
-			(effects
-				(font
-					(size 1.27 1.27)
-				)
-			)
-		)
-		(property "Description" "Power symbol creates a global label with name \"GND\" , ground"
-			(at 166.37 158.75 0)
-			(hide yes)
-			(show_name no)
-			(do_not_autoplace no)
-			(effects
-				(font
-					(size 1.27 1.27)
-				)
-			)
-		)
-		(pin "1"
-		)
-		(instances
-			(project "version2"
-				(path "/accd8c2f-694c-41c7-8115-13b6db3d60fb"
-					(reference "#PWR019")
-					(unit 1)
-				)
-			)
-		)
-	)
-	(symbol
 		(lib_id "Device:R")
 		(at 180.34 148.59 180)
@@
 					(unit 1)
 				)
-			)
-		)
-	)
-	(symbol
-		(lib_id "power:GND")
-		(at 166.37 200.66 0)
-		(unit 1)
-		(body_style 1)
-		(exclude_from_sim no)
-		(in_bom yes)
-		(on_board yes)
-		(in_pos_files yes)
-		(dnp no)
-		(fields_autoplaced yes)
-		(property "Reference" "#PWR023"
-			(at 166.37 207.01 0)
-			(hide yes)
-			(show_name no)
-			(do_not_autoplace no)
-			(effects
-				(font
-					(size 1.27 1.27)
-				)
-			)
-		)
-		(property "Value" "GND"
-			(at 166.37 205.74 0)
-			(show_name no)
-			(do_not_autoplace no)
-			(effects
-				(font
-					(size 1.27 1.27)
-				)
-			)
-		)
-		(property "Footprint" ""
-			(at 166.37 200.66 0)
-			(hide yes)
-			(show_name no)
-			(do_not_autoplace no)
-			(effects
-				(font
-					(size 1.27 1.27)
-				)
-			)
-		)
-		(property "Datasheet" ""
-			(at 166.37 200.66 0)
-			(hide yes)
-			(show_name no)
-			(do_not_autoplace no)
-			(effects
-				(font
-					(size 1.27 1.27)
-				)
-			)
-		)
-		(property "Description" "Power symbol creates a global label with name \"GND\" , ground"
-			(at 166.37 200.66 0)
-			(hide yes)
-			(show_name no)
-			(do_not_autoplace no)
-			(effects
-				(font
-					(size 1.27 1.27)
-				)
-			)
-		)
-		(pin "1"
-		)
-		(instances
-			(project "version2"
-				(path "/accd8c2f-694c-41c7-8115-13b6db3d60fb"
-					(reference "#PWR023")
-					(unit 1)
-				)

Commit message: edited mounting holes
Parts:
- added H1, H2, H3, H4: MountingHole, symbol Mechanical:MountingHole
